File: ESP12Module.kicad_pcb (KiCad board)
At the start: 2 copper layers, 44.5 x 31.8 mm, 19 parts, among them J1 Conn_01x05_Male, J2 Conn_01x05_Male, J3 Screw_Terminal_01x02, J4 Conn_01x02_Male, SW4 SW_Push, U2 ESP-12S, sw3 SW_Push

Commit message: Add files via upload
Parts:
- removed sw3: SW_Push, Button_Switch_THT:SW_PUSH_6mm
- added SW3: SW_Push, Button_Switch_THT:SW_PUSH_6mm, F.Cu at (80.5, 76.8)
Connections:
- J1 pad 2: /Rx -> /Tx
- J1 pad 3: /Tx -> /Rx
- R1 pad 1: /Rx -> /Tx
- R2 pad 1: /Tx -> /Rx
- U2 pad 15: /Tx -> /Rx
- U2 pad 16: /Rx -> /Tx
Routing:
- net /RST: track 54.4 -> 40.1 mm, vias 2 -> 4
- net VCC: track 22.2 -> 34.2 mm, vias 8 -> 10
- net /Tx: track 18.0 -> 11.7 mm
- net /Rx: track 11.7 -> 18.0 mm
- net GND: track 51.1 -> 56.0 mm, vias 1 -> 2
- net /PIN0: track 106.6 -> 103.8 mm
- net /PIN15: track 41.9 -> 39.5 mm
- net /PIN13: track 46.6 -> 44.7 mm
- net (no net): track 1.44 -> 0.00 mm
- net Net-(D1-Pad2): track 33.9 -> 32.8 mm
- net Net-(D2-Pad2): track 39.0 -> 38.4 mm
Other:
- board text added: "."
- board text added: "Version 1.0"
