File: ESP12Module.sch (KiCad schematic (older format))
At the start: 19 parts, among them J1 Conn_01x05_Male, J2 Conn_01x05_Male, J3 Screw_Terminal_01x02, J4 Conn_01x02_Male, SW4 SW_Push, U2 ESP-12S, sw3 SW_Push

Commit message: Add files via upload
Parts:
- renumbered sw3 to SW3
Connections:
- net Rx: now also J1.3 (Pin_3), R2.1, U2.15 (RXD0); no longer J1.2 (Pin_2), R1.1, U2.16 (TXD0)
- net Tx: now also J1.2 (Pin_2), R1.1, U2.16 (TXD0); no longer J1.3 (Pin_3), R2.1, U2.15 (RXD0)
Other:
- moved on the sheet: C4, D1, D2, J1, J2, J3, J4, R1, R10, R11, R12, R13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
